Commit message: PG Chopstick: finger sleeves with record buttons, colour bimanual robot renders, chopstick-only README
- Handheld jaws get finger sleeves (sleeve.py): Ø20 ring under the dotted shelf, 5.5 mm pad with a 6x6 switch
  pocket, domed TPU cover and wire channel; jaw_right_dc split from the robot's jaw_right
- Button roles by jaw: right-jaw sleeve (right hand index) = start/stop, left-jaw sleeve (left hand index) = cancel;
  pod gets two wire entries, docs and firmware notes updated
- ISO 50 plate default roll flipped so the camera is on top with the usual tool0 convention
- robots.py: UR5, ABB GoFa and FANUC CRX dual-arm renders in their own colours, PG Chopsticks on both flanges,
  poses from a small IK
- Root README is now the in-depth PG Chopstick README (sync_readme.py), with a bimanual UR5 example

File: chopstick/urdf/pg_chopstick_data.urdf (robot description, URDF)
Before this commit: robot pg_chopstick_data, 7 links, 6 joints
Links:
- link chopstick_base: mass 0.27139 -> 0.27136
- link chopstick_jaw_left: mass 0.048789 -> 0.053445; geometry collision mesh filename=meshes/jaw_left_dc_jawframe.stl scale=0.001 0.001 0.001; collision mesh filename=meshes/sleeve_button_cover_left_jawframe.stl scale=0.001 0.001 0.001
- link chopstick_jaw_right: mass 0.048723 -> 0.05338; geometry collision mesh filename=meshes/jaw_right_dc_jawframe.stl scale=0.001 0.001 0.001; collision mesh filename=meshes/sleeve_button_cover_right_jawframe.stl scale=0.001 0.001 0.001

File: chopstick/urdf/pg_chopstick_data_d405.urdf (robot description, URDF)
Before this commit: robot pg_chopstick_data_d405, 7 links, 6 joints
Links:
- link chopstick_jaw_left: mass 0.048789 -> 0.053445; geometry collision mesh filename=meshes/jaw_left_dc_jawframe.stl scale=0.001 0.001 0.001; collision mesh filename=meshes/sleeve_button_cover_left_jawframe.stl scale=0.001 0.001 0.001
- link chopstick_jaw_right: mass 0.048723 -> 0.05338; geometry collision mesh filename=meshes/jaw_right_dc_jawframe.stl scale=0.001 0.001 0.001; collision mesh filename=meshes/sleeve_button_cover_right_jawframe.stl scale=0.001 0.001 0.001

File: chopstick/urdf/pg_chopstick_iso50.urdf (robot description, URDF)
Before this commit: robot pg_chopstick_iso50, 8 links, 7 joints
Joints:
- joint chopstick_mount_joint: origin xyz=0 0 0.016 rpy=3.14159265 -1.57079633 0 -> xyz=0 0 0.016 rpy=0 -1.57079633 0

File: chopstick/urdf/pg_chopstick_iso50_d405.urdf (robot description, URDF)
Before this commit: robot pg_chopstick_iso50_d405, 8 links, 7 joints
Joints:
- joint chopstick_mount_joint: origin xyz=0 0 0.016 rpy=3.14159265 -1.57079633 0 -> xyz=0 0 0.016 rpy=0 -1.57079633 0
