Commit message: WIP checkpoint: elastic finger straps, D405 on the HandUMI tilt hinge, clean FANUC renders, parallel-jaw first pass
- Finger sleeves: printed pad + two strap fins with slots for an elastic hook-and-loop strap; one record button,
  in the index-finger jaw only (data_right: start/stop, data_left: cancel); pod button removed
- D405 frame: HandUMI D405 cup on a Ø12 / M4 centre knuckle, tilts 15-65 deg clear of everything, top cable window
- robots.py: FANUC from two clean CRX-5iA arms side by side, same layout and IK as the UR / ABB renders
- parallel.py: first pass of a rack-and-pinion parallel gripper on the X5 frame (parts only; not yet
  clash-checked or integrated into the builds, URDFs or docs)

File: chopstick/urdf/pg_chopstick_data_d405.urdf (robot description, URDF)
Before this commit: robot pg_chopstick_data_d405, 7 links, 6 joints
Links:
- link chopstick_jaw_left: mass 0.053445 -> 0.054642; geometry collision mesh filename=meshes/jaw_left_dc_jawframe.stl scale=0.001 0.001 0.001; collision mesh filename=meshes/sleeve_strap_left_jawframe.stl scale=0.001 0.001 0.001
- link chopstick_jaw_right: mass 0.05338 -> 0.054576; geometry collision mesh filename=meshes/jaw_right_dc_jawframe.stl scale=0.001 0.001 0.001; collision mesh filename=meshes/sleeve_strap_right_jawframe.stl scale=0.001 0.001 0.001

File: chopstick/urdf/pg_chopstick_data_left.urdf (robot description, URDF)
Before this commit: robot pg_chopstick_data, 7 links, 6 joints
Links:
- link chopstick_base: mass 0.27136 -> 0.27072; geometry collision mesh filename=meshes/chopstick_base_dc.stl scale=0.001 0.001 0.001; collision mesh filename=meshes/chopstick_clip_dc.stl scale=0.001 0.001 0.001
- link chopstick_jaw_left: mass 0.053445 -> 0.054547; geometry collision mesh filename=meshes/jaw_left_dc_button_jawframe.stl scale=0.001 0.001 0.001; collision mesh filename=meshes/sleeve_button_cover_left_jawframe.stl scale=0.001 0.001 0.001
- link chopstick_jaw_right: mass 0.05338 -> 0.054576; geometry collision mesh filename=meshes/jaw_right_dc_jawframe.stl scale=0.001 0.001 0.001; collision mesh filename=meshes/sleeve_strap_right_jawframe.stl scale=0.001 0.001 0.001
