Commit message: D405 parallel = HandUMI as-is; real Quest Touch Pro controller; realistic hand and robot-hand renders
Synced from pg-chopstick: cad/d405 and assembly/d405. The parallel gripper is HandUMI unchanged (vendored in
cad/d405/handumi, built by t_gripper.py, no interferences at any opening with any tip set). The cradle now holds Meta's
Touch Pro controller model (file git-ignored). The hand render shows a posed hand and forearm with the strap, and
hand_robot.png the same head on a Shadow Hand on a UR5e. README and video updated.

File: assembly/d405/chopstick/urdf/pg_chopstick_left.urdf (robot description, URDF)
Before this commit: robot pg_chopstick_left, 7 links, 6 joints
Links:
- link pg_base: mass 0.29945 -> 0.33745

File: assembly/d405/chopstick/urdf/pg_chopstick_right.urdf (robot description, URDF)
Before this commit: robot pg_chopstick_right, 7 links, 6 joints
Links:
- link pg_base: mass 0.29945 -> 0.33745

File: assembly/d405/hand/urdf/pg_hand.urdf (robot description, URDF)
Before this commit: robot pg_hand, 2 links, 1 joints
Links:
- link pg_base: mass 0.3198 -> 0.3578
