Commit message: Chop-UMI / Para-UMI names; thumb strap and palm button on the hand build; robot camera posts for Para-UMI; FANUC render fix; HandUMI controller support for the Quest (face forward, mirrored), stiffer D405 frame

File: assembly/d405/hand/urdf/pg_hand.urdf (robot description, URDF)
Before this commit: robot pg_hand, 2 links, 1 joints
Links:
- link pg_base: mass 0.3578 -> 0.34166; geometry collision mesh filename=meshes/d405_cup.stl scale=0.001 0.001 0.001; collision mesh filename=meshes/d405_envelope.stl scale=0.001 0.001 0.001
