Commit message: Main: render gallery README; PG Chopstick as Chop-UMI / Para-UMI / Hand with the Quest in HandUMI's support, thumb strap and palm button, robot camera posts

File: pg-chopstick/insta360_x5/hand/urdf/pg_hand.urdf (robot description, URDF)
Before this commit: robot pg_hand, 2 links, 1 joints
Links:
- link pg_base: mass 0.28235 -> 0.2831
